Commit message: 220624-3

File: ip50_description/urdf/ip50.urdf.xacro (robot description, xacro)
@@ -169,5 +169,5 @@
     <parent link="center_link"/>
     <child link="lidar_link"/>
-    <origin xyz="0.2511 0 0.017" rpy="0 0 0"/>
+    <origin xyz="0.2511 0 0.017" rpy="0 0 ${-PI/2}"/>
   </joint>
   <!-- The diff between  0.2m -->
